File: KiCad/Schematics/June0.0.1/KeyWordFinal.kicad_sch (KiCad schematic)
At the start: 36 parts, among them J1 ${ALTIUM_VALUE}, J2 Conn_01x05_Pin, J6 ${ALTIUM_VALUE}, U1 ${ALTIUM_VALUE}, U2 ${ALTIUM_VALUE}, U3 TPS627431YFPR, U4 TXB0104D, X1 ${ALTIUM_VALUE}, X2 ${ALTIUM_VALUE}

Commit message: Added all components to schematic
Parts:
- added J3: Micro_SD_Card, symbol Connector:Micro_SD_Card
- added MK1: 3SM123GZB1VE-R, 3SM123GZB1VE-R:MIC_3SM123GZB1VE-R, symbol 3SM123GZB1VE-R:3SM123GZB1VE-R
- added P1: USB_C_Plug_USB2.0, symbol Connector:USB_C_Plug_USB2.0
- added U5: Opamp_Dual, symbol Amplifier_Operational:Opamp_Dual
Connections:
- net GND: now also J3.6 (VSS), J3.SH (SHIELD), MK1.3_1 (GND), MK1.3_2 (GND__1), U5.4 (V-)
- net VHIGH: now also J3.4 (VDD)
- net VLOW: now also MK1.1 (VDD), U5.8 (V+)
- net at U4.10 (B4): now also J3.7 (DAT0)
- net at U4.11 (B3): now also J3.5 (CLK)
- net at U4.12 (B2): now also J3.3 (CMD)
- net at U4.13 (B1): now also J3.2 (DAT3/CD)
- new net: P1.A1 (GND), P1.A12 (GND), P1.B1 (GND), P1.B12 (GND)
- new net: P1.A4 (VBUS), P1.A9 (VBUS), P1.B4 (VBUS), P1.B9 (VBUS)
- no-connect marks 0 -> 2
Other:
- note added: "1 extra GPIO, maybe detection LED?"
- note added: "ADC input + and -"

Commit message: Finished wiring schematic
Parts:
- added C18, C19, C20: ${ALTIUM_VALUE}, CAPC1608X06L, symbol AltiumLib:CAP
- added D3: LED, symbol Device:LED
- added R1, R10, R11, R2, R3, R4, R5, R6, R7, R8, R9, R_CC: ${ALTIUM_VALUE}, RESC0603X03L_C, symbol AltiumLib:RES
Connections:
- net GND: now also P1.A1 (GND), P1.A12 (GND), P1.A7 (D-), P1.B1 (GND), P1.B12 (GND), P1.SH (SHIELD), C19.1, C20.1, R2.1, R8.1, R9.1, R_CC.1
- net P0.04/AIN2: now also U5.3 (+), U5.5 (+), R7.1, R8.2
- net P0.05/AIN3: now also C20.2, R11.1
- net P0.14: now also D3.2 (A)
- net VBUS: now also P1.A4 (VBUS), P1.A9 (VBUS), P1.B4 (VBUS), P1.B9 (VBUS)
- net VLOW: now also R1.2, R7.2
- net at U5.6 (-): now also R5.1, R6.2
- net at U5.7: now also R10.2, R6.1
- net at P1.A5 (CC): now also R_CC.2
- net at MK1.2 (OUTPUT): now also C18.2
- net at U5.1: now also R4.1, R5.2
- net at U5.2 (-): now also R3.1, R4.2
- new net: D3.1 (K), R9.2
- new net: C18.1, R1.1, R2.2, R3.2
- new net: C19.2, R10.1, R11.2
- no-connect marks 2 -> 5
Other:
- moved on the sheet: J1, P1, U5A, U5B, U5C
