File: KiCad/Schematics+Layout/June0.1.0/KeyWordFinal.kicad_sch (KiCad schematic)
At the start: 54 parts, among them J1 USB4105-GF-A, J2 Conn_01x02_Pin, J3 Conn_01x05_Pin, J4 MSD-10-C, U1 NRF52805-CAAA-R, U2 NPM1100-CAAA-R7, U3 TXB0104RUTR, U4 TPS62743YFPR, U5 MCP6142T-E/MS, Y1 32.768k, Y3 32M

Commit message: Combine schematics and layout
Parts:
- added AE1: Antenna_Chip, RF_Antenna:Texas_SWRA117D_2.4GHz_Left, symbol Device:Antenna_Chip
- added C23, C24, C25, C26, C28: 0.1u, Capacitor_SMD:C_0603_1608Metric, symbol Device:C
- added C27: 1.0u, Capacitor_SMD:C_0603_1608Metric, symbol Device:C
- C19: value C -> 10n
- R6, R7: value R -> 100k
Connections:
- net +1V8: now also C23.2, C24.2, C25.2
- net +3V0: now also C26.2, C27.1, C28.1
- net GND: now also AE1.2 (PCB_Trace), C23.1, C24.1, C25.1, C26.1, C27.2, C28.2
- net RF: now also AE1.1 (FEED)
- no-connect marks 6 -> 5

Commit message: Updated layout, updated schematic to ease layout.
Connections:
- net +1V8: now also U3.12 (OE); no longer U3.8 (OE)
- net +3V0: now also U3.11 (VCCB); no longer U3.14 (VCCB)
- net ADC+: now also U1.F5 (P0.04/AIN2); no longer U1.F6 (P0.05/AIN3)
- net GND: now also U3.6 (GND); no longer U3.7 (GND)
- net VCOM: now also U1.F6 (P0.05/AIN3); no longer U1.F5 (P0.04/AIN2)
- net at C16.2, U1.A1 (XC1): now also Y3.3; no longer Y3.1
- net at J4.05 (CLK): now also U3.9 (B2); no longer U3.11 (B3)
- net at J4.03 (CMD): now also U3.8 (B3); no longer U3.12 (B2)
- net at J4.02 (DAT3/CD): now also U3.7 (B4); no longer U3.13 (B1)
- net at U3.2 (A1): now also U1.G5 (P0.12); no longer U1.F2 (P0.20)
- net at U3.3 (A2): now also U1.G4 (P0.16); no longer U1.G3 (P0.18)
- net at U3.4 (A3): now also U1.G3 (P0.18); no longer U1.G4 (P0.16)
- net at U3.5 (A4): now also U1.F4 (P0.14); no longer U1.G5 (P0.12)
- net at C17.2, U1.A2 (XC2): now also Y3.1; no longer Y3.3
- net at D3.2 (A): now also U1.F2 (P0.20); no longer U1.F4 (P0.14)
Other:
- moved on the sheet: C26
Changed lines of the file:
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@@
 	)
 	(junction
-		(at 160.02 115.57)
+		(at 160.02 151.13)
 		(diameter 0)
 		(color 0 0 0 0)
@@
 	)
 	(junction
+		(at 147.32 147.32)
+		(diameter 0)
+		(color 0 0 0 0)
+	)
+	(junction
 		(at 231.14 68.58)
 		(diameter 0)
@@
 	)
 	(junction
-		(at 154.94 115.57)
+		(at 154.94 151.13)
 		(diameter 0)
 		(color 0 0 0 0)
@@
 	)
 	(junction
-		(at 147.32 120.65)
-		(diameter 0)
-		(color 0 0 0 0)
-	)
-	(junction
 		(at 27.94 151.13)
 		(diameter 0)
@@
 	(wire
 		(pts
-			(xy 146.05 120.65) (xy 147.32 120.65)
+			(xy 146.05 147.32) (xy 147.32 147.32)
 		)
 		(stroke
@@
 	(wire
 		(pts
-			(xy 118.11 138.43) (xy 118.11 146.05)
-		)
-		(stroke
-			(width 0)
-			(type default)
-		)
-	)
-	(wire
-		(pts
 			(xy 231.14 59.69) (xy 231.14 60.96)
 		)
@@
 	(wire
 		(pts
-			(xy 105.41 125.73) (xy 147.32 125.73)
+			(xy 105.41 125.73) (xy 116.84 125.73)
 		)
 		(stroke
@@
 	(wire
 		(pts
-			(xy 146.05 147.32) (xy 146.05 120.65)
-		)
-		(stroke
-			(width 0)
-			(type default)
-		)
-	)
-	(wire
-		(pts
 			(xy 204.47 20.32) (xy 195.58 20.32)
 		)
@@
 	(wire
 		(pts
-			(xy 147.32 120.65) (xy 147.32 115.57)
+			(xy 147.32 146.05) (xy 147.32 147.32)
 		)
 		(stroke
@@
 	(wire
 		(pts
+			(xy 118.11 125.73) (xy 118.11 138.43)
+		)
+		(stroke
+			(width 0)
+			(type default)
+		)
+	)
+	(wire
+		(pts
 			(xy 107.95 45.72) (xy 110.49 45.72)
 		)
@@
 	(wire
 		(pts
-			(xy 147.32 115.57) (xy 154.94 115.57)
+			(xy 147.32 151.13) (xy 154.94 151.13)
 		)
 		(stroke
@@
 	(wire
 		(pts
+			(xy 147.32 147.32) (xy 147.32 151.13)
+		)
+		(stroke
+			(width 0)
+			(type default)
+		)
+	)
+	(wire
+		(pts
 			(xy 171.45 30.48) (xy 171.45 33.02)
 		)
@@
 	(wire
 		(pts
+			(xy 118.11 125.73) (xy 147.32 125.73)
+		)
+		(stroke
+			(width 0)
+			(type default)
+		)
+	)
+	(wire
+		(pts
 			(xy 80.01 107.95) (xy 80.01 102.87)
 		)
@@
 	(wire
 		(pts
-			(xy 118.11 146.05) (xy 134.62 146.05)
+			(xy 116.84 146.05) (xy 134.62 146.05)
 		)
 		(stroke
@@
 	(wire
 		(pts
+			(xy 116.84 146.05) (xy 116.84 125.73)
+		)
+		(stroke
+			(width 0)
+			(type default)
+		)
+	)
+	(wire
+		(pts
 			(xy 107.95 55.88) (xy 107.95 54.61)
 		)
@@
 		)
 	)
-	(label "ADC-"
+	(label "ADC+"
 		(at 130.81 176.53 0)
 		(effects
@@
 		)
 	)
-	(label "ADC+"
+	(label "ADC-"
 		(at 130.81 173.99 0)
 		(effects
@@
 	(symbol
 		(lib_id "power:+1V8")
-		(at 154.94 115.57 0)
+		(at 154.94 151.13 0)
+		(mirror x)
 		(unit 1)
 		(body_style 1)
@@
 		(fields_autoplaced yes)
 		(property "Reference" "#PWR034"
-			(at 154.94 119.38 0)
+			(at 154.94 147.32 0)
 			(hide yes)
 			(show_name no)
@@
 		)
 		(property "Value" "+1V8"
-			(at 154.94 110.49 0)
+			(at 154.94 156.21 0)
 			(show_name no)
 			(do_not_autoplace no)
@@
 		)
 		(property "Footprint" ""
-			(at 154.94 115.57 0)
+			(at 154.94 151.13 0)
 			(hide yes)
 			(show_name no)
@@
 		)
 		(property "Datasheet" ""
-			(at 154.94 115.57 0)
+			(at 154.94 151.13 0)
 			(hide yes)
 			(show_name no)
@@
 		)
 		(property "Description" "Power symbol creates a global label with name \"+1V8\""
-			(at 154.94 115.57 0)
+			(at 154.94 151.13 0)
 			(hide yes)
 			(show_name no)
@@
 		(lib_id "ProjSyms:TXB0104RUTR")
 		(at 157.48 133.35 0)
+		(mirror x)
 		(unit 1)
 		(body_style 1)
@@
 		(fields_autoplaced yes)
 		(property "Reference" "U3"
-			(at 187.96 123.19 0)
+			(at 187.96 143.51 0)
 			(hide yes)
 			(show_name no)
@@
 		)
 		(property "Value" "TXB0104RUTR"
-			(at 187.96 125.73 0)
+			(at 187.96 140.97 0)
 			(hide yes)
 			(show_name no)
@@
 		(pin "11"
 		)
-		(pin "13"
+		(pin "9"
 		)
-		(pin "14"
+		(pin "6"
 		)
 		(pin "12"
@@
 	(symbol
 		(lib_id "power:GND")
-		(at 157.48 151.13 0)
+		(at 157.48 115.57 0)
+		(mirror x)
 		(unit 1)
 		(body_style 1)
@@
 		(fields_autoplaced yes)
 		(property "Reference" "#PWR035"
-			(at 157.48 157.48 0)
+			(at 157.48 109.22 0)
 			(hide yes)
 			(show_name no)
@@
 		)
 		(property "Value" "GND"
-			(at 157.48 156.21 0)
+			(at 157.48 110.49 0)
 			(show_name no)
 			(do_not_autoplace no)
@@
 		)
 		(property "Footprint" ""
-			(at 157.48 151.13 0)
+			(at 157.48 115.57 0)
 			(hide yes)
 			(show_name no)
@@
 		)
 		(property "Datasheet" ""
-			(at 157.48 151.13 0)
+			(at 157.48 115.57 0)
 			(hide yes)
 			(show_name no)
@@
 		)
 		(property "Description" "Power symbol creates a global label with name \"GND\" , ground"
-			(at 157.48 151.13 0)
+			(at 157.48 115.57 0)
 			(hide yes)
 			(show_name no)
@@
 	(symbol
 		(lib_id "power:GND")
-		(at 167.64 115.57 0)
+		(at 167.64 151.13 0)
+		(mirror x)
 		(unit 1)
 		(body_style 1)
@@
 		(fields_autoplaced yes)
 		(property "Reference" "#PWR059"
-			(at 167.64 121.92 0)
+			(at 167.64 144.78 0)
 			(hide yes)
 			(show_name no)
@@
 		)
 		(property "Value" "GND"
-			(at 167.64 120.65 0)
+			(at 167.64 146.05 0)
 			(show_name no)
 			(do_not_autoplace no)
@@
 		)
 		(property "Footprint" ""
-			(at 167.64 115.57 0)
+			(at 167.64 151.13 0)
 			(hide yes)
 			(show_name no)
@@
 		)
 		(property "Datasheet" ""
-			(at 167.64 115.57 0)
+			(at 167.64 151.13 0)
 			(hide yes)
 			(show_name no)
@@
 		)
 		(property "Description" "Power symbol creates a global label with name \"GND\" , ground"
-			(at 167.64 115.57 0)
+			(at 167.64 151.13 0)
 			(hide yes)
 			(show_name no)
@@
 	(symbol
 		(lib_id "power:+3V0")
-		(at 160.02 115.57 0)
+		(at 160.02 151.13 0)
+		(mirror x)
 		(unit 1)
 		(body_style 1)
@@
 		(fields_autoplaced yes)
 		(property "Reference" "#PWR026"
-			(at 160.02 119.38 0)
+			(at 160.02 147.32 0)
 			(hide yes)
 			(show_name no)
@@
 		)
 		(property "Value" "+3V0"
-			(at 160.02 110.49 0)
+			(at 160.02 156.21 0)
 			(show_name no)
 			(do_not_autoplace no)
@@
 		)
 		(property "Footprint" ""
-			(at 160.02 115.57 0)
+			(at 160.02 151.13 0)
 			(hide yes)
 			(show_name no)
@@
 		)
 		(property "Datasheet" ""
-			(at 160.02 115.57 0)
+			(at 160.02 151.13 0)
 			(hide yes)
 			(show_name no)
@@
 		)
 		(property "Description" "Power symbol creates a global label with name \"+3V0\""
-			(at 160.02 115.57 0)
+			(at 160.02 151.13 0)
 			(hide yes)
 			(show_name no)
@@
 		(in_pos_files yes)
 		(dnp no)
-		(fields_autoplaced yes)
 		(property "Reference" "C25"
-			(at 149.86 149.8599 0)
+			(at 149.86 152.3999 0)
 			(show_name no)
 			(do_not_autoplace no)
@@
 		)
 		(property "Value" "0.1u"
-			(at 149.86 152.3999 0)
+			(at 149.86 154.9399 0)
 			(show_name no)
 			(do_not_autoplace no)
@@
 		(lib_id "Device:Crystal_GND24")
 		(at 55.88 101.6 270)
+		(mirror x)
 		(unit 1)
 		(body_style 1)
@@
 		(in_pos_files yes)
 		(dnp no)
-		(fields_autoplaced yes)
 		(property "Reference" "Y3"
-			(at 60.96 100.3299 90)
+			(at 60.96 102.8701 90)
 			(show_name no)
 			(do_not_autoplace no)
@@
 		)
 		(property "Value" "32M"
-			(at 60.96 102.8699 90)
+			(at 60.96 100.3301 90)
 			(show_name no)
 			(do_not_autoplace no)
@@
 	(symbol
 		(lib_id "Device:C")
-		(at 163.83 115.57 270)
+		(at 163.83 151.13 270)
+		(mirror x)
 		(unit 1)
 		(body_style 1)
@@
 		(fields_autoplaced yes)
 		(property "Reference" "C26"
-			(at 163.83 107.95 90)
+			(at 163.83 158.75 90)
 			(show_name no)
 			(do_not_autoplace no)
@@
 		)
 		(property "Value" "0.1u"
-			(at 163.83 110.49 90)
+			(at 163.83 156.21 90)
 			(show_name no)
 			(do_not_autoplace no)
@@
 		)
 		(property "Footprint" "Capacitor_SMD:C_0603_1608Metric"
-			(at 160.02 116.5352 0)
+			(at 160.02 150.1648 0)
 			(hide yes)
 			(show_name no)
@@
 		)
 		(property "Datasheet" ""
-			(at 163.83 115.57 0)
+			(at 163.83 151.13 0)
 			(hide yes)
 			(show_name no)
@@
 		)
 		(property "Description" "Unpolarized capacitor"
-			(at 163.83 115.57 0)
+			(at 163.83 151.13 0)
 			(hide yes)
 			(show_name no)

Commit message: Added some traces to test placement
Parts:
- R6: footprint Resistor_SMD:R_0402_1005Metric -> Resistor_SMD:R_0603_1608Metric
Connections:
- net VBUS: now also C12.1, U4.A2 (VIN), U4.B1 (EN), U4.D1 (VSEL2), U4.D2 (VSEL3)
- net V_{INT}: no longer C12.1, U4.A2 (VIN), U4.B1 (EN), U4.D1 (VSEL2), U4.D2 (VSEL3)
- net at U3.9 (B2): now also J4.05 (CLK)
Changed lines of the file:
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@@
 	)
 	(junction
+		(at 220.98 22.86)
+		(diameter 0)
+		(color 0 0 0 0)
+	)
+	(junction
 		(at 262.89 35.56)
 		(diameter 0)
@@
 	)
 	(junction
-		(at 220.98 22.86)
-		(diameter 0)
-		(color 0 0 0 0)
-	)
-	(junction
 		(at 229.87 22.86)
 		(diameter 0)
@@
 	)
 	(symbol
-		(lib_id "power:VINT")
-		(at 220.98 22.86 0)
-		(unit 1)
-		(body_style 1)
-		(exclude_from_sim no)
-		(in_bom yes)
-		(on_board yes)
-		(in_pos_files yes)
-		(dnp no)
-		(fields_autoplaced yes)
-		(property "Reference" "#PWR042"
-			(at 220.98 26.67 0)
-			(hide yes)
-			(show_name no)
-			(do_not_autoplace no)
-			(effects
-				(font
-					(size 1.27 1.27)
-				)
-			)
-		)
-		(property "Value" "V_{INT}"
-			(at 220.98 17.78 0)
-			(show_name no)
-			(do_not_autoplace no)
-			(effects
-				(font
-					(size 1.27 1.27)
-				)
-			)
-		)
-		(property "Footprint" ""
-			(at 220.98 22.86 0)
-			(hide yes)
-			(show_name no)
-			(do_not_autoplace no)
-			(effects
-				(font
-					(size 1.27 1.27)
-				)
-			)
-		)
-		(property "Datasheet" ""
-			(at 220.98 22.86 0)
-			(hide yes)
-			(show_name no)
-			(do_not_autoplace no)
-			(effects
-				(font
-					(size 1.27 1.27)
-				)
-			)
-		)
-		(property "Description" "Power symbol creates a global label with name \"VINT\""
-			(at 220.98 22.86 0)
-			(hide yes)
-			(show_name no)
-			(do_not_autoplace no)
-			(effects
-				(font
-					(size 1.27 1.27)
-				)
-			)
-		)
-		(pin "1"
-		)
-		(instances
-			(project "KeyWordFinal"
-				(path "/f9fa5162-c43b-4303-9827-e483132d8026"
-					(reference "#PWR042")
-					(unit 1)
-				)
-			)
-		)
-	)
-	(symbol
 		(lib_id "power:+3V0")
 		(at 271.78 22.86 270)
@@
 	)
 	(symbol
+		(lib_id "power:VBUS")
+		(at 220.98 22.86 0)
+		(unit 1)
+		(body_style 1)
+		(exclude_from_sim no)
+		(in_bom yes)
+		(on_board yes)
+		(in_pos_files yes)
+		(dnp no)
+		(fields_autoplaced yes)
+		(property "Reference" "#PWR057"
+			(at 220.98 26.67 0)
+			(hide yes)
+			(show_name no)
+			(do_not_autoplace no)
+			(effects
+				(font
+					(size 1.27 1.27)
+				)
+			)
+		)
+		(property "Value" "VBUS"
+			(at 220.98 17.78 0)
+			(show_name no)
+			(do_not_autoplace no)
+			(effects
+				(font
+					(size 1.27 1.27)
+				)
+			)
+		)
+		(property "Footprint" ""
+			(at 220.98 22.86 0)
+			(hide yes)
+			(show_name no)
+			(do_not_autoplace no)
+			(effects
+				(font
+					(size 1.27 1.27)
+				)
+			)
+		)
+		(property "Datasheet" ""
+			(at 220.98 22.86 0)
+			(hide yes)
+			(show_name no)
+			(do_not_autoplace no)
+			(effects
+				(font
+					(size 1.27 1.27)
+				)
+			)
+		)
+		(property "Description" "Power symbol creates a global label with name \"VBUS\""
+			(at 220.98 22.86 0)
+			(hide yes)
+			(show_name no)
+			(do_not_autoplace no)
+			(effects
+				(font
+					(size 1.27 1.27)
+				)
+			)
+		)
+		(pin "1"
+		)
+		(instances
+			(project "KeyWordFinal"
+				(path "/f9fa5162-c43b-4303-9827-e483132d8026"
+					(reference "#PWR057")
+					(unit 1)
+				)
+			)
+		)
+	)
+	(symbol
 		(lib_id "power:+1V8")
 		(at 132.08 99.06 0)
@@
 			)
 		)
-		(property "Footprint" "Resistor_SMD:R_0402_1005Metric"
+		(property "Footprint" "Resistor_SMD:R_0603_1608Metric"
 			(at 229.362 54.61 90)
 			(hide yes)
